Commit message: SM thesis code arrangement

File: src/ObjectDetection/models/urdf/cube.urdf (robot description, URDF)
Before this commit: robot cube, 1 links, 0 joints
Links:
- link cube_1: geometry collision box size=1.00 1.00 1.00; visual box size=1.00 1.00 1.00

File: src/ObjectDetection/models/urdf/cubes.urdf (robot description, URDF)
Before this commit: robot cube, 2 links, 0 joints
Links:
- link cube_1: geometry collision box size=1.0 1.0 1.0; visual box size=1.0 1.0 1.0
- link cube_2: geometry collision box size=2.0 1.0 1.0; visual box size=2.0 1.0 1.0
