Commit message: updated urdf for better ik

File: models/ur10/ur10_description/ur10_robot_half.urdf (robot description, URDF)
Before this commit: robot ur10, 13 links, 12 joints
Joints:
- joint elbow_joint: limit lower=-3.1431853 upper=3.1431853 effort=150.0 velocity=3.15 -> lower=-3.1431853 upper=3.1431853 effort=1.0 velocity=3.15
- joint shoulder_lift_joint: limit lower=-3.1431853 upper=3.1431853 effort=330.0 velocity=2.16 -> lower=-3.1431853 upper=3.1431853 effort=1.0 velocity=2.16
- joint shoulder_pan_joint: limit lower=-3.1431853 upper=3.1431853 effort=330.0 velocity=2.16 -> lower=-3.1431853 upper=3.1431853 effort=1.0 velocity=2.16
- joint wrist_1_joint: limit lower=-3.1431853 upper=3.1431853 effort=54.0 velocity=3.2 -> lower=-3.1431853 upper=3.1431853 effort=1.0 velocity=3.2
- joint wrist_2_joint: limit lower=-3.1431853 upper=3.1431853 effort=54.0 velocity=3.2 -> lower=-3.1431853 upper=3.1431853 effort=1.0 velocity=3.2
- joint wrist_3_joint: limit lower=-3.1431853 upper=3.1431853 effort=54.0 velocity=3.2 -> lower=-3.1431853 upper=3.1431853 effort=1.0 velocity=3.2
