Commit message: Update models to match Drake's iiwa14 models

File: models/iiwa/iiwa_description/iiwa14.urdf (robot description, URDF)
Before this commit: robot iiwa14, 11 links, 10 joints
Links:
- link iiwa_link_0: geometry collision cylinder length=0.17 radius=0.139; visual mesh filename=package://iiwa_description/meshes/visual/link_0.obj
- link iiwa_link_1: geometry collision cylinder length=0.29 radius=0.101; visual mesh filename=package://iiwa_description/meshes/visual/link_1.obj
- link iiwa_link_2: geometry collision cylinder length=0.29 radius=0.101; visual mesh filename=package://iiwa_description/meshes/visual/link_2_grey.obj
- link iiwa_link_3: geometry collision cylinder length=0.29 radius=0.092; visual mesh filename=package://iiwa_description/meshes/visual/band.obj
- link iiwa_link_4: geometry collision cylinder length=0.25 radius=0.092; visual mesh filename=package://iiwa_description/meshes/visual/link_4_grey.obj
- link iiwa_link_5: geometry collision cylinder length=0.29 radius=0.07; visual mesh filename=package://iiwa_description/meshes/visual/band.obj
- link iiwa_link_6: geometry collision mesh filename=package://iiwa_description/meshes/collision/link_6.obj; visual mesh filename=package://iiwa_description/meshes/visual/link_6_grey.obj
- link iiwa_link_7: geometry collision mesh filename=meshes/collision/link_7.obj; visual mesh filename=package://iiwa_description/meshes/visual/link_7.obj
Joints:
- removed joint base_joint
- added joint iiwa_base_joint: type fixed, parent base, child iiwa_link_0, origin xyz=0 0 0 rpy=0 0 0
- joint iiwa_joint_2: origin xyz=0 0 0.2025 rpy=1.57079632679   0 3.14159265359 -> xyz=0 0 0.2025 rpy=1.570796326794897   0 3.141592653589793
- joint iiwa_joint_3: origin xyz=0 0.2045 0 rpy=1.57079632679 0 3.14159265359 -> xyz=0 0.2045 0 rpy=1.570796326794897 0 3.141592653589793
- joint iiwa_joint_4: origin xyz=0 0 0.2155 rpy=1.57079632679 0 0 -> xyz=0 0 0.2155 rpy=1.570796326794897 0 0
- joint iiwa_joint_5: origin xyz=0 0.1845 0 rpy=-1.57079632679 3.14159265359 0 -> xyz=0 0.1845 0 rpy=-1.570796326794897 3.141592653589793 0
- joint iiwa_joint_6: origin xyz=0 0 0.2155 rpy=1.57079632679 0 0 -> xyz=0 0 0.2155 rpy=1.570796326794897 0 0
- joint iiwa_joint_7: origin xyz=0 0.081 0 rpy=-1.57079632679 3.14159265359 0 -> xyz=0 0.081 0 rpy=-1.570796326794897 3.141592653589793 0
- joint iiwa_joint_ee: origin xyz=0 0 0.045 rpy=3.14159265359 3.14159265359 3.14159265359 -> xyz=0 0 0.045 rpy=3.141592653589793 3.141592653589793 3.141592653589793
- joint tool0_joint: origin xyz=0 0 0.045 rpy=0 -1.57079632679 0 -> xyz=0 0 0.045 rpy=0 -1.570796326794897 0

File: models/iiwa/iiwa_description/iiwa14_schunk_gripper.urdf (robot description, URDF)
Before this commit: robot iiwa14, 18 links, 17 joints
Links:
- link iiwa_link_1: mass 4 -> 5.76
- link iiwa_link_2: mass 4 -> 6.35; geometry collision cylinder length=0.29 radius=0.101; visual mesh filename=package://iiwa_description/meshes/visual/link_2_grey.obj
- link iiwa_link_3: mass 3 -> 3.5; geometry collision cylinder length=0.29 radius=0.092; visual mesh filename=package://iiwa_description/meshes/visual/band.obj
- link iiwa_link_4: mass 2.7 -> 3.5; geometry collision cylinder length=0.25 radius=0.092; visual mesh filename=package://iiwa_description/meshes/visual/link_4_grey.obj
- link iiwa_link_5: mass 1.7 -> 3.5; geometry collision cylinder length=0.29 radius=0.07; visual mesh filename=package://iiwa_description/meshes/visual/band.obj
- link iiwa_link_6: geometry collision mesh filename=meshes/collision/link_6.obj; visual mesh filename=package://iiwa_description/meshes/visual/link_6_grey.obj
- link iiwa_link_7: mass 0.3 -> 1.2; geometry collision mesh filename=meshes/collision/link_7.obj; visual mesh filename=package://iiwa_description/meshes/visual/link_7.obj
Joints:
- removed joint base_joint
- added joint iiwa_base_joint: type fixed, parent base, child iiwa_link_0, origin xyz=0 0 0 rpy=0 0 0
- joint iiwa_joint_2: origin xyz=0 0 0.2025 rpy=1.57079632679   0 3.14159265359 -> xyz=0 0 0.2025 rpy=1.570796326794897   0 3.141592653589793
- joint iiwa_joint_3: origin xyz=0 0.2045 0 rpy=1.57079632679 0 3.14159265359 -> xyz=0 0.2045 0 rpy=1.570796326794897 0 3.141592653589793
- joint iiwa_joint_4: origin xyz=0 0 0.2155 rpy=1.57079632679 0 0 -> xyz=0 0 0.2155 rpy=1.570796326794897 0 0
- joint iiwa_joint_5: origin xyz=0 0.1845 0 rpy=-1.57079632679 3.14159265359 0 -> xyz=0 0.1845 0 rpy=-1.570796326794897 3.141592653589793 0
- joint iiwa_joint_6: origin xyz=0 0 0.2155 rpy=1.57079632679 0 0 -> xyz=0 0 0.2155 rpy=1.570796326794897 0 0
- joint iiwa_joint_7: origin xyz=0 0.081 0 rpy=-1.57079632679 3.14159265359 0 -> xyz=0 0.081 0 rpy=-1.570796326794897 3.141592653589793 0
- joint iiwa_joint_ee: origin xyz=0 0 0.045 rpy=3.14159265359 3.14159265359 3.14159265359 -> xyz=0 0 0.045 rpy=3.141592653589793 3.141592653589793 3.141592653589793
- joint tool0_joint: origin xyz=0 0 0.045 rpy=0 -1.57079632679 0 -> xyz=0 0 0.045 rpy=0 -1.570796326794897 0

File: models/iiwa/iiwa_description/iiwa14_schunk_gripper_drake_sim.urdf (robot description, URDF)
Before this commit: robot iiwa14, 17 links, 16 joints
Links:
- link iiwa_link_0: geometry collision cylinder length=0.17 radius=0.139; visual mesh filename=package://iiwa_description/meshes/visual/link_0.obj
- link iiwa_link_1: mass 4 -> 5.76; geometry collision cylinder length=0.29 radius=0.101; visual mesh filename=package://iiwa_description/meshes/visual/link_1.obj
- link iiwa_link_2: mass 4 -> 6.35; geometry collision cylinder length=0.29 radius=0.101; visual mesh filename=package://iiwa_description/meshes/visual/link_2_grey.obj
- link iiwa_link_3: mass 3 -> 3.5; geometry collision cylinder length=0.29 radius=0.092; visual mesh filename=package://iiwa_description/meshes/visual/band.obj
- link iiwa_link_4: mass 2.7 -> 3.5; geometry collision cylinder length=0.25 radius=0.092; visual mesh filename=package://iiwa_description/meshes/visual/link_4_grey.obj
- link iiwa_link_5: mass 1.7 -> 3.5; geometry collision cylinder length=0.29 radius=0.07; visual mesh filename=package://iiwa_description/meshes/visual/band.obj
- link iiwa_link_6: geometry collision mesh filename=meshes/collision/link_6.obj; visual mesh filename=package://iiwa_description/meshes/visual/link_6_grey.obj
- link iiwa_link_7: mass 0.3 -> 1.2; geometry collision mesh filename=meshes/collision/link_7.obj; visual mesh filename=package://iiwa_description/meshes/visual/link_7.obj
Joints:
- removed joint base_joint
- added joint iiwa_base_joint: type fixed, parent base, child iiwa_link_0, origin xyz=0 0 0 rpy=0 0 0
- joint iiwa_joint_2: origin xyz=0 0 0.2025 rpy=1.57079632679   0 3.14159265359 -> xyz=0 0 0.2025 rpy=1.570796326794897   0 3.141592653589793
- joint iiwa_joint_3: origin xyz=0 0.2045 0 rpy=1.57079632679 0 3.14159265359 -> xyz=0 0.2045 0 rpy=1.570796326794897 0 3.141592653589793
- joint iiwa_joint_4: origin xyz=0 0 0.2155 rpy=1.57079632679 0 0 -> xyz=0 0 0.2155 rpy=1.570796326794897 0 0
- joint iiwa_joint_5: origin xyz=0 0.1845 0 rpy=-1.57079632679 3.14159265359 0 -> xyz=0 0.1845 0 rpy=-1.570796326794897 3.141592653589793 0
- joint iiwa_joint_6: origin xyz=0 0 0.2155 rpy=1.57079632679 0 0 -> xyz=0 0 0.2155 rpy=1.570796326794897 0 0
- joint iiwa_joint_7: origin xyz=0 0.081 0 rpy=-1.57079632679 3.14159265359 0 -> xyz=0 0.081 0 rpy=-1.570796326794897 3.141592653589793 0
- joint iiwa_joint_ee: origin xyz=0 0 0.045 rpy=3.14159265359 3.14159265359 3.14159265359 -> xyz=0 0 0.045 rpy=3.141592653589793 3.141592653589793 3.141592653589793
- joint tool0_joint: origin xyz=0 0 0.045 rpy=0 -1.57079632679 0 -> xyz=0 0 0.045 rpy=0 -1.570796326794897 0

File: models/iiwa/iiwa_description/iiwa14_simplified_collision.urdf (robot description, URDF)
Before this commit: robot iiwa14, 11 links, 10 joints
Links:
- link iiwa_link_0: geometry visual mesh filename=package://iiwa_description/meshes/visual/link_0.obj
- link iiwa_link_1: geometry visual mesh filename=package://iiwa_description/meshes/visual/link_1.obj
- link iiwa_link_2: geometry visual mesh filename=package://iiwa_description/meshes/visual/link_2_grey.obj; visual mesh filename=package://iiwa_description/meshes/visual/link_2_orange.obj
- link iiwa_link_3: geometry visual mesh filename=package://iiwa_description/meshes/visual/band.obj; visual mesh filename=package://iiwa_description/meshes/visual/kuka.obj
- link iiwa_link_4: geometry visual mesh filename=package://iiwa_description/meshes/visual/link_4_grey.obj; visual mesh filename=package://iiwa_description/meshes/visual/link_4_orange.obj
- link iiwa_link_5: geometry visual mesh filename=package://iiwa_description/meshes/visual/band.obj; visual mesh filename=package://iiwa_description/meshes/visual/kuka.obj
- link iiwa_link_6: geometry visual mesh filename=package://iiwa_description/meshes/visual/link_6_grey.obj; visual mesh filename=package://iiwa_description/meshes/visual/link_6_orange.obj
- link iiwa_link_7: geometry collision mesh filename=meshes/collision/link_7_polytope.obj; visual mesh filename=package://iiwa_description/meshes/visual/link_7.obj
Joints:
- removed joint base_joint
- added joint iiwa_base_joint: type fixed, parent base, child iiwa_link_0, origin xyz=0 0 0 rpy=0 0 0
- joint iiwa_joint_2: origin xyz=0 0 0.2025 rpy=1.57079632679   0 3.14159265359 -> xyz=0 0 0.2025 rpy=1.570796326794897   0 3.141592653589793
- joint iiwa_joint_3: origin xyz=0 0.2045 0 rpy=1.57079632679 0 3.14159265359 -> xyz=0 0.2045 0 rpy=1.570796326794897 0 3.141592653589793
- joint iiwa_joint_4: origin xyz=0 0 0.2155 rpy=1.57079632679 0 0 -> xyz=0 0 0.2155 rpy=1.570796326794897 0 0
- joint iiwa_joint_5: origin xyz=0 0.1845 0 rpy=-1.57079632679 3.14159265359 0 -> xyz=0 0.1845 0 rpy=-1.570796326794897 3.141592653589793 0
- joint iiwa_joint_6: origin xyz=0 0 0.2155 rpy=1.57079632679 0 0 -> xyz=0 0 0.2155 rpy=1.570796326794897 0 0
- joint iiwa_joint_7: origin xyz=0 0.081 0 rpy=-1.57079632679 3.14159265359 0 -> xyz=0 0.081 0 rpy=-1.570796326794897 3.141592653589793 0
- joint iiwa_joint_ee: origin xyz=0 0 0.045 rpy=3.14159265359 3.14159265359 3.14159265359 -> xyz=0 0 0.045 rpy=3.141592653589793 3.141592653589793 3.141592653589793
- joint tool0_joint: origin xyz=0 0 0.045 rpy=0 -1.57079632679 0 -> xyz=0 0 0.045 rpy=0 -1.570796326794897 0
