Commit message: Mostly rely on Drake for the iiwa description meshes Removes duplicated meshes (and whole urdfs) in favor of relying on drake's versions. Exception is a URDF that glues together the iiwa and schunk gripper, which we will keep a copy of. This will probably be slightly adjusted as we modify our iiwa setup, but it makes sense to duplicate as few of these meshes as possible?

File: models/iiwa/iiwa_description/iiwa14_schunk_gripper.urdf (robot description, URDF)
Before this commit: robot iiwa14, 14 links, 13 joints
Links:
- removed link palm
- removed link wsg_50_finger_left_link
- removed link wsg_50_finger_right_link
- added link wsg_50_base_link, mass 1.2; collision mesh filename=package://wsg_50_description/meshes/WSG50_110.obj scale=1 1 1; visual mesh filename=package://wsg_50_description/meshes/WSG50_110.obj scale=1 1 1
- added link wsg_50_finger_left, mass 0.1; collision mesh filename=package://wsg_50_description/meshes/WSG-FMF.obj scale=0.001 0.001 0.001; visual mesh filename=package://wsg_50_description/meshes/WSG-FMF.obj scale=0.001 0.001 0.001
- added link wsg_50_finger_right, mass 0.1; collision mesh filename=package://wsg_50_description/meshes/WSG-FMF.obj scale=0.001 0.001 0.001; visual mesh filename=package://wsg_50_description/meshes/WSG-FMF.obj scale=0.001 0.001 0.001
- added link wsg_50_gripper_left, mass 0.1; collision mesh filename=package://wsg_50_description/meshes/GUIDE_WSG50_110.obj scale=0.001 0.001 0.001; visual mesh filename=package://wsg_50_description/meshes/GUIDE_WSG50_110.obj scale=0.001 0.001 0.001
- added link wsg_50_gripper_right, mass 0.1; collision mesh filename=package://wsg_50_description/meshes/GUIDE_WSG50_110.obj scale=0.001 0.001 0.001; visual mesh filename=package://wsg_50_description/meshes/GUIDE_WSG50_110.obj scale=0.001 0.001 0.001
- link iiwa_link_0: geometry visual mesh filename=package://iiwa_description/meshes/visual/link_0.obj
- link iiwa_link_1: mass 4 -> 5.76; geometry visual mesh filename=package://iiwa_description/meshes/visual/link_1.obj
- link iiwa_link_2: mass 4 -> 6.35; geometry visual mesh filename=package://iiwa_description/meshes/visual/link_2.obj
- link iiwa_link_3: mass 3 -> 3.5; geometry visual mesh filename=package://iiwa_description/meshes/visual/link_3.obj
- link iiwa_link_4: mass 2.7 -> 3.5; geometry visual mesh filename=package://iiwa_description/meshes/visual/link_4.obj
- link iiwa_link_5: mass 1.7 -> 3.5; geometry visual mesh filename=package://iiwa_description/meshes/visual/link_5.obj
- link iiwa_link_7: mass 0.3 -> 1.2; geometry collision mesh filename=package://iiwa_description/meshes/collision/link_7_polytope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; visual mesh filename=package://iiwa_description/meshes/visual/link_7.obj
Joints:
- removed joint base_joint
- removed joint gripper_mount_joint
- removed joint wsg_50_finger_left_joint
- removed joint wsg_50_finger_right_joint
- added joint iiwa_base_joint: type fixed, parent base, child iiwa_link_0, origin xyz=0 0 0 rpy=0 0 0
- added joint wsg_50_base_joint_gripper_left: type prismatic, parent wsg_50_base_link, child wsg_50_gripper_left, origin xyz=0 0 0 rpy=0 0 0, axis 1 0 0, limit lower=-0.055 upper=-0.0027 effort=1.0 velocity=1.0
- added joint wsg_50_base_joint_gripper_right: type prismatic, parent wsg_50_base_link, child wsg_50_gripper_right, origin xyz=0 0 0 rpy=0 0 3.14159, axis -1 0 0, limit lower=0.0027 upper=0.055 effort=1.0 velocity=1.0
- added joint wsg_50_guide_joint_finger_left: type fixed, parent wsg_50_gripper_left, child wsg_50_finger_left, origin xyz=0 0 0.023 rpy=0 0 0, axis 1 0 0, limit effort=100 velocity=100
- added joint wsg_50_guide_joint_finger_right: type fixed, parent wsg_50_gripper_right, child wsg_50_finger_right, origin xyz=0 0 0.023 rpy=0 0 0, axis 1 0 0, limit effort=100 velocity=100
- added joint wsg_50_mount_joint: type fixed, parent iiwa_link_ee, child wsg_50_base_link, origin xyz=0.005 0 0 rpy=1.57079632679 0 1.57079632679, axis 0 0 1

Commit message: Mostly rely on Drake for the iiwa description meshes Removes duplicated meshes (and whole urdfs) in favor of relying on drake's versions. Exception is a URDF that glues together the iiwa and schunk gripper, which we will keep a copy of. This will probably be slightly adjusted as we modify our iiwa setup, but it makes sense to duplicate as few of these meshes as possible?

File: models/iiwa/iiwa_description/iiwa14_schunk_gripper.urdf (robot description, URDF)
Before this commit: robot iiwa14, 14 links, 13 joints
Links:
- removed link palm
- removed link wsg_50_finger_left_link
- removed link wsg_50_finger_right_link
- added link wsg_50_base_link, mass 1.2; collision mesh filename=package://wsg_50_description/meshes/WSG50_110.obj scale=1 1 1; visual mesh filename=package://wsg_50_description/meshes/WSG50_110.obj scale=1 1 1
- added link wsg_50_finger_left, mass 0.1; collision mesh filename=package://wsg_50_description/meshes/WSG-FMF.obj scale=0.001 0.001 0.001; visual mesh filename=package://wsg_50_description/meshes/WSG-FMF.obj scale=0.001 0.001 0.001
- added link wsg_50_finger_right, mass 0.1; collision mesh filename=package://wsg_50_description/meshes/WSG-FMF.obj scale=0.001 0.001 0.001; visual mesh filename=package://wsg_50_description/meshes/WSG-FMF.obj scale=0.001 0.001 0.001
- added link wsg_50_gripper_left, mass 0.1; collision mesh filename=package://wsg_50_description/meshes/GUIDE_WSG50_110.obj scale=0.001 0.001 0.001; visual mesh filename=package://wsg_50_description/meshes/GUIDE_WSG50_110.obj scale=0.001 0.001 0.001
- added link wsg_50_gripper_right, mass 0.1; collision mesh filename=package://wsg_50_description/meshes/GUIDE_WSG50_110.obj scale=0.001 0.001 0.001; visual mesh filename=package://wsg_50_description/meshes/GUIDE_WSG50_110.obj scale=0.001 0.001 0.001
- link iiwa_link_0: geometry visual mesh filename=package://iiwa_description/meshes/visual/link_0.obj
- link iiwa_link_1: mass 4 -> 5.76; geometry visual mesh filename=package://iiwa_description/meshes/visual/link_1.obj
- link iiwa_link_2: mass 4 -> 6.35; geometry visual mesh filename=package://iiwa_description/meshes/visual/link_2.obj
- link iiwa_link_3: mass 3 -> 3.5; geometry visual mesh filename=package://iiwa_description/meshes/visual/link_3.obj
- link iiwa_link_4: mass 2.7 -> 3.5; geometry visual mesh filename=package://iiwa_description/meshes/visual/link_4.obj
- link iiwa_link_5: mass 1.7 -> 3.5; geometry visual mesh filename=package://iiwa_description/meshes/visual/link_5.obj
- link iiwa_link_6: geometry visual mesh filename=package://iiwa_description/meshes/visual/link_6.obj
- link iiwa_link_7: mass 0.3 -> 1.2; geometry collision mesh filename=package://iiwa_description/meshes/collision/link_7_polytope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; visual mesh filename=package://iiwa_description/meshes/visual/link_7.obj
Joints:
- removed joint base_joint
- removed joint gripper_mount_joint
- removed joint wsg_50_finger_left_joint
- removed joint wsg_50_finger_right_joint
- added joint iiwa_base_joint: type fixed, parent base, child iiwa_link_0, origin xyz=0 0 0 rpy=0 0 0
- added joint wsg_50_base_joint_gripper_left: type prismatic, parent wsg_50_base_link, child wsg_50_gripper_left, origin xyz=0 0 0 rpy=0 0 0, axis 1 0 0, limit lower=-0.055 upper=-0.0027 effort=1.0 velocity=1.0
- added joint wsg_50_base_joint_gripper_right: type prismatic, parent wsg_50_base_link, child wsg_50_gripper_right, origin xyz=0 0 0 rpy=0 0 3.14159, axis -1 0 0, limit lower=0.0027 upper=0.055 effort=1.0 velocity=1.0
- added joint wsg_50_guide_joint_finger_left: type fixed, parent wsg_50_gripper_left, child wsg_50_finger_left, origin xyz=0 0 0.023 rpy=0 0 0, axis 1 0 0, limit effort=100 velocity=100
- added joint wsg_50_guide_joint_finger_right: type fixed, parent wsg_50_gripper_right, child wsg_50_finger_right, origin xyz=0 0 0.023 rpy=0 0 0, axis 1 0 0, limit effort=100 velocity=100
- added joint wsg_50_mount_joint: type fixed, parent iiwa_link_ee, child wsg_50_base_link, origin xyz=0.005 0 0 rpy=1.57079632679 0 1.57079632679, axis 0 0 1

Commit message: Modify iiwa schunk gripper paths for rviz rendering

File: models/iiwa/iiwa_description/iiwa14_schunk_gripper.urdf (robot description, URDF)
Before this commit: robot iiwa14, 14 links, 13 joints
Links:
- link iiwa_link_0: geometry collision cylinder length=0.17 radius=0.139; visual mesh filename=package://iiwa_description/meshes/visual/link_0.obj
- link iiwa_link_1: geometry collision cylinder length=0.29 radius=0.101; visual mesh filename=package://iiwa_description/meshes/visual/link_1.obj
- link iiwa_link_2: geometry collision cylinder length=0.29 radius=0.101; visual mesh filename=package://iiwa_description/meshes/visual/link_2.obj
- link iiwa_link_3: geometry collision cylinder length=0.29 radius=0.092; visual mesh filename=package://iiwa_description/meshes/visual/link_3.obj
- link iiwa_link_4: geometry collision cylinder length=0.25 radius=0.092; visual mesh filename=package://iiwa_description/meshes/visual/link_4.obj
- link iiwa_link_5: geometry collision cylinder length=0.29 radius=0.07; visual mesh filename=package://iiwa_description/meshes/visual/link_5.obj
- link iiwa_link_6: geometry collision mesh filename=package://iiwa_description/meshes/collision/link_6.obj; visual mesh filename=package://iiwa_description/meshes/visual/link_6.obj
- link iiwa_link_7: geometry collision mesh filename=package://iiwa_description/meshes/collision/link_7.obj; visual mesh filename=package://iiwa_description/meshes/visual/link_7.obj
Joints:
- joint wsg_50_finger_left_joint: limit (none) -> lower=-0.001 upper=0.109 effort=10 velocity=1.0
- joint wsg_50_finger_right_joint: limit (none) -> lower=-0.001 upper=0.109 effort=10 velocity=1.0

Commit message: Fix missing collision mesh paths and fix bullet sim

File: models/iiwa/iiwa_description/iiwa14_schunk_gripper.urdf (robot description, URDF)
Before this commit: robot iiwa14, 18 links, 17 joints
Links:
- link iiwa_link_6: geometry collision mesh filename=package://iiwa_description/meshes/collision/link_6.obj; visual mesh filename=package://iiwa_description/meshes/visual/link_6_grey.obj
- link iiwa_link_7: geometry collision mesh filename=package://iiwa_description/meshes/collision/link_7.obj; visual mesh filename=package://iiwa_description/meshes/visual/link_7.obj
