Commit message: peg in hole sim now working

File: src/catkin_projects/drake_iiwa_sim/models/square_peg_receptacle.xacro (robot description, xacro)
@@ -3,6 +3,6 @@
 <xacro:property name="x_dim_outer" value="0.3" />
 <xacro:property name="y_dim_outer" value="0.3" />
-<xacro:property name="x_dim_inner" value="0.075" />
-<xacro:property name="y_dim_inner" value="0.1" />
+<xacro:property name="x_dim_inner" value="0.05" />
+<xacro:property name="y_dim_inner" value="0.05" />
 <xacro:property name="z_dim" value="0.05" />
 <!-- macro for making default inertial mass-->
